Commit message: Update jdcobot_100_description.urdf

File: urdf/jdcobot_100_description.urdf (robot description, URDF)
Before this commit: robot jdcobot_100_description, 7 links, 6 joints
Joints:
- joint joint_1: limit lower=0 upper=0 effort=0 velocity=0 -> lower=0 upper=3.1416 effort=0 velocity=0
- joint joint_2: limit lower=0 upper=0 effort=0 velocity=0 -> lower=0 upper=3.1416 effort=0 velocity=0
- joint joint_3: limit lower=0 upper=0 effort=0 velocity=0 -> lower=0 upper=3.1416 effort=0 velocity=0
- joint joint_4: limit lower=0 upper=0 effort=0 velocity=0 -> lower=0 upper=3.1416 effort=0 velocity=0
- joint joint_5: limit lower=0 upper=0 effort=0 velocity=0 -> lower=0 upper=3.1416 effort=0 velocity=0
- joint joint_6: mimic joint=joint_5 multiplier=1 offset=0 -> joint=joint_5 multiplier=0.05 offset=0; origin xyz=-0.007818 0.063831 0.010521 rpy=0 3.1416 1.5708 -> xyz=-0.007818 0.063831 0.1562 rpy=0 3.1416 1.5708

Commit message: Update jdcobot_100_description.urdf

File: urdf/jdcobot_100_description.urdf (robot description, URDF)
Before this commit: robot jdcobot_100_description, 7 links, 6 joints
Joints:
- joint joint_6: limit lower=0 upper=0.03 effort=0 velocity=0 -> lower=0.001 upper=0.003 effort=0 velocity=0; mimic joint=joint_5 multiplier=0.05 offset=0 -> joint=joint_5 multiplier=0.0062 offset=0; origin xyz=-0.007818 0.063831 0.1562 rpy=0 3.1416 1.5708 -> xyz=-0.007818 0.063831 0.018 rpy=0 3.1416 1.5708
